File: PCB/Macropad.kicad_pcb (KiCad board)
At the start: 2 copper layers, 6 parts, among them SW1 SW_Push, SW2 SW_Push, SW3 SW_Push, SW4 SW_Push, SW5 RotaryEncoder_Switch, U1 XIAO-RP2040-DIP

Commit message: Add files via upload
Routing:
- net Net-(U1-GPIO28/ADC2/A2): track 0.00 -> 67.8 mm, vias 0 -> 4
- net GND: track 89.6 -> 140.5 mm, vias 0 -> 2
Changed lines of the file:
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@@
+	)
+	(segment
+		(start 154.684375 90.584375)
+		(end 158.601 94.501)
+		(width 0.2)
+		(layer "F.Cu")
+		(net 1)
 	)
 	(segment
@@
 	)
 	(segment
+		(start 176.199 84.303)
+		(end 176.199 78.56775)
+		(width 0.2)
+		(layer "F.Cu")
+		(net 1)
+	)
+	(segment
 		(start 149.86 109.22)
 		(end 149.86 90.17)
@@
 	)
 	(segment
+		(start 176.199 78.56775)
+		(end 173.83125 76.2)
+		(width 0.2)
+		(layer "F.Cu")
+		(net 1)
+	)
+	(segment
+		(start 158.601 94.501)
+		(end 166.001 94.501)
+		(width 0.2)
+		(layer "F.Cu")
+		(net 1)
+	)
+	(segment
 		(start 174.3 93.2)
 		(end 171.8 95.7)
@@
 	)
 	(segment
+		(start 171.45 69.05625)
+		(end 170.71375 68.32)
+		(width 0.2)
+		(layer "F.Cu")
+		(net 1)
+	)
+	(segment
+		(start 170.71375 68.32)
+		(end 165.455 68.32)
+		(width 0.2)
+		(layer "F.Cu")
+		(net 1)
+	)
+	(segment
 		(start 149.86 128.27)
 		(end 149.86 109.22)
@@
 	(segment
 		(start 159.8 95.7)
+		(end 154.684375 90.584375)
+		(width 0.2)
+		(layer "F.Cu")
+		(net 1)
+	)
+	(segment
+		(start 166.001 94.501)
+		(end 176.199 84.303)
+		(width 0.2)
+		(layer "F.Cu")
+		(net 1)
+	)
+	(segment
+		(start 154.684375 90.584375)
 		(end 154.27 90.17)
 		(width 0.2)
@@
 		(net 1)
 	)
+	(via
+		(at 171.45 69.05625)
+		(size 0.6)
+		(drill 0.3)
+		(layers "F.Cu" "B.Cu")
+		(net 1)
+	)
+	(via
+		(at 173.83125 76.2)
+		(size 0.6)
+		(drill 0.3)
+		(layers "F.Cu" "B.Cu")
+		(net 1)
+	)
+	(segment
+		(start 171.45 73.81875)
+		(end 171.45 69.05625)
+		(width 0.2)
+		(layer "B.Cu")
+		(net 1)
+	)
+	(segment
+		(start 173.83125 76.2)
+		(end 171.45 73.81875)
+		(width 0.2)
+		(layer "B.Cu")
+		(net 1)
+	)
 	(segment
 		(start 169.2275 118.9275)
@@
 	)
 	(segment
+		(start 145.83375 70.86)
+		(end 148.545 70.86)
+		(width 0.2)
+		(layer "F.Cu")
+		(net 5)
+	)
+	(segment
+		(start 142.875 71.4375)
+		(end 145.25625 71.4375)
+		(width 0.2)
+		(layer "F.Cu")
+		(net 5)
+	)
+	(segment
+		(start 159.8 93.2)
+		(end 166.6875 86.3125)
+		(width 0.2)
+		(layer "F.Cu")
+		(net 5)
+	)
+	(segment
+		(start 145.25625 71.4375)
+		(end 145.83375 70.86)
+		(width 0.2)
+		(layer "F.Cu")
+		(net 5)
+	)
+	(segment
+		(start 166.6875 86.3125)
+		(end 166.6875 85.7)
+		(width 0.2)
+		(layer "F.Cu")
+		(net 5)
+	)
+	(segment
+		(start 169.06875 79.08)
+		(end 169.06875 76.54)
+		(width 0.2)
+		(layer "F.Cu")
+		(net 5)
+	)
+	(via
+		(at 169.06875 79.08)
+		(size 0.6)
+		(drill 0.3)
+		(layers "F.Cu" "B.Cu")
+		(net 5)
+	)
+	(via
+		(at 169.06875 76.54)
+		(size 0.6)
+		(drill 0.3)
+		(layers "F.Cu" "B.Cu")
+		(net 5)
+	)
+	(via
+		(at 142.875 71.4375)
+		(size 0.6)
+		(drill 0.3)
+		(layers "F.Cu" "B.Cu")
+		(net 5)
+	)
+	(via
+		(at 166.6875 85.7)
+		(size 0.6)
+		(drill 0.3)
+		(layers "F.Cu" "B.Cu")
+		(net 5)
+	)
+	(segment
+		(start 166.6875 85.7)
+		(end 169.06875 83.31875)
+		(width 0.2)
+		(layer "B.Cu")
+		(net 5)
+	)
+	(segment
+		(start 142.875 69.05625)
+		(end 142.875 71.4375)
+		(width 0.2)
+		(layer "B.Cu")
+		(net 5)
+	)
+	(segment
+		(start 169.06875 83.31875)
+		(end 169.06875 79.08)
+		(width 0.2)
+		(layer "B.Cu")
+		(net 5)
+	)
+	(segment
+		(start 145.25625 66.675)
+		(end 142.875 69.05625)
+		(width 0.2)
+		(layer "B.Cu")
+		(net 5)
+	)
+	(segment
+		(start 169.06875 66.675)
+		(end 166.6875 64.29375)
+		(width 0.2)
+		(layer "B.Cu")
+		(net 5)
+	)
+	(segment
+		(start 147.6375 64.29375)
+		(end 145.25625 66.675)
+		(width 0.2)
+		(layer "B.Cu")
+		(net 5)
+	)
+	(segment
+		(start 169.06875 76.54)
+		(end 169.06875 66.675)
+		(width 0.2)
+		(layer "B.Cu")
+		(net 5)
+	)
+	(segment
+		(start 166.6875 64.29375)
+		(end 147.6375 64.29375)
+		(width 0.2)
+		(layer "B.Cu")
+		(net 5)
+	)
+	(segment
